Commit message: fix: 进一步缩小底盘碰撞半径防止轮子嵌套
问题分析:
- 轮距: 0.3420 m (固定参数)
- 轮子半径: 0.0632 m (固定参数)
- 轮子内沿: 0.171 - 0.0632 = 0.1078 m
- 之前碰撞半径: 0.15 m → 轮子还是嵌在底盘里

修复:
- 碰撞半径: 0.15 m → 0.10 m
- 现在: 0.1078 m > 0.10 m → 轮子不会嵌入底盘

验证方法:
重启roslaunch后检查Gazebo中轮子是否与底盘分离

Co-Authored-By: Claude Sonnet 4.5 <noreply@anthropic.com>

File: catkin_ws/src/dashgo_rl/urdf/dashgo_d1_sim.urdf.xacro (robot description, xacro)
@@ -48,5 +48,5 @@
       <origin xyz="0 0 0" rpy="0 0 0"/>
       <geometry>
-        <cylinder length="0.21" radius="0.15"/>  <!-- 0.20 → 0.15 防止轮子穿模 -->
+        <cylinder length="0.21" radius="0.10"/>  <!-- 0.15 → 0.10 进一步缩小以避免轮子嵌在底盘里 -->
       </geometry>
     </collision>

Commit message: fix: 抬高底盘碰撞体避免拖底(方案A)
问题诊断(Isaac Sim架构师):
- 底盘碰撞体太大太低，先着地把轮子架空
- 旧配置: origin z=0, length=0.21, radius=0.10
- 底盘底部: z=-0.105m, 轮子底部: z=-0.0632m
- 结论: 底盘先着地，轮子悬空 ❌

修复方案(方案A-保守):
- origin xyz: "0 0 0" → "0 0 0.05" (向上抬高5cm)
- length: 0.21 → 0.10 (厚度减半)
- radius: 保持0.10 (避免水平方向碰撞轮子)

新几何验证:
- 底盘中心: z=0.05m, 厚度=0.10m
- 底盘底部: 0.05 - 0.05 = 0.00m
- 轮子底部: -0.0632m
- 结论: 轮子先着地(0.00 > -0.0632) ✅

水平方向验证:
- 轮子内沿: 0.1078m
- 底盘半径: 0.10m
- 结论: 不会水平碰撞(0.10 < 0.1078) ✅

相关commit:
- ffed4ef: 调整spawn高度到0.0632(轮子半径)

Co-Authored-By: Claude Sonnet 4.5 <noreply@anthropic.com>

File: catkin_ws/src/dashgo_rl/urdf/dashgo_d1_sim.urdf.xacro (robot description, xacro)
@@ -46,7 +46,7 @@
     </visual>
     <collision>
-      <origin xyz="0 0 0" rpy="0 0 0"/>
+      <origin xyz="0 0 0.05" rpy="0 0 0"/>
       <geometry>
-        <cylinder length="0.21" radius="0.10"/>  <!-- 0.15 → 0.10 进一步缩小以避免轮子嵌在底盘里 -->
+        <cylinder length="0.10" radius="0.10"/>  <!-- 抬高5cm避免拖底，厚度减半，半径保持0.10避免水平碰撞 -->
       </geometry>
     </collision>

Commit message: feat: 修复重心位置并添加万向轮(Dashgo D1实机参数)
问题1: 小车倾斜
原因: inertial重心在z=0，collision碰撞体在z=0.05
      → 重心太低，碰撞体太高 → 头重脚轻
修复: inertial添加origin xyz="0 0 0.05" (跟随碰撞体)

问题2: 小车稳定性差（缺少支撑）
实机参数: Dashgo D1采用1+2+1布局（前万向+中驱动+后万向）
        - 底盘直径: 406mm
        - 离地高度: 38mm
        - 自重: 20kg

实现:
1. 添加前万向轮(front_caster_link)
   - 位置: (0.15, 0, -0.05) - 底盘前方
   - 半径: 12.7mm (1寸万向轮)
   - 质量: 0.1kg

2. 添加后万向轮(rear_caster_link)
   - 位置: (-0.15, 0, -0.05) - 底盘后方
   - 半径: 12.7mm (1寸万向轮)
   - 质量: 0.1kg

3. 万向轮摩擦力属性
   - mu1=0.0, mu2=0.0 (低摩擦便于转向)
   - 驱动轮保持mu1=1.0, mu2=1.0

验证:
重启roslaunch后检查:
1. 小车不再倾斜（重心与碰撞体对齐）
2. 4个轮子着地（前万向+2驱动+后万向）
3. 稳定性提升，不会侧翻

参考文档:
- dashgo/EAI驱动/dashgo_bringup/config/my_dashgo_params.yaml

Co-Authored-By: Claude Sonnet 4.5 <noreply@anthropic.com>

File: catkin_ws/src/dashgo_rl/urdf/dashgo_d1_sim.urdf.xacro (robot description, xacro)
@@ -52,4 +52,5 @@
     </collision>
     <inertial>
+      <origin xyz="0 0 0.05" rpy="0 0 0"/>  <!-- 🔥 修复：重心跟随碰撞体 -->
       <mass value="${base_mass}"/>
       <inertia ixx="0.05" ixy="0" ixz="0" iyy="0.05" iyz="0" izz="0.08"/>
@@ -57,5 +58,67 @@
   </link>
   <!-- =========================================================
-       轮子定义
+       万向轮定义（Caster Wheels）- Dashgo D1实机参数
+       布局：1+2+1（前万向 + 中驱动 + 后万向）
+    ========================================================== -->
+  <xacro:property name="caster_radius" value="0.0127"/>   <!-- 1寸万向轮半径=12.7mm -->
+  <xacro:property name="caster_mass" value="0.1"/>           <!-- 万向轮质量 -->
+  <!-- 前万向轮 -->
+  <link name="front_caster_link">
+    <visual>
+      <geometry>
+        <sphere radius="${caster_radius}"/>
+      </geometry>
+      <origin rpy="0 0 0" xyz="0 0 0"/>
+      <material name="gray">
+        <color rgba="0.5 0.5 0.5 1.0"/>
+      </material>
+    </visual>
+    <collision>
+      <geometry>
+        <sphere radius="${caster_radius}"/>
+      </geometry>
+      <origin rpy="0 0 0" xyz="0 0 0"/>
+    </collision>
+    <inertial>
+      <mass value="${caster_mass}"/>
+      <inertia ixx="0.00001" ixy="0" ixz="0" iyy="0.00001" iyz="0" izz="0.00001"/>
+    </inertial>
+  </link>
+  <joint name="front_caster_joint" type="fixed">
+    <parent link="base_link"/>
+    <child link="front_caster_link"/>
+    <!-- 前万向轮位置：底盘前方（假设1+2+1布局，前后对称） -->
+    <origin xyz="0.15 0 -0.05" rpy="0 0 0"/>
+  </joint>
+  <!-- 后万向轮 -->
+  <link name="rear_caster_link">
+    <visual>
+      <geometry>
+        <sphere radius="${caster_radius}"/>
+      </geometry>
+      <origin rpy="0 0 0" xyz="0 0 0"/>
+      <material name="gray">
+        <color rgba="0.5 0.5 0.5 1.0"/>
+      </material>
+    </visual>
+    <collision>
+      <geometry>
+        <sphere radius="${caster_radius}"/>
+      </geometry>
+      <origin rpy="0 0 0" xyz="0 0 0"/>
+    </collision>
+    <inertial>
+      <mass value="${caster_mass}"/>
+      <inertia ixx="0.00001" ixy="0" ixz="0" iyy="0.00001" iyz="0" izz="0.00001"/>
+    </inertial>
+  </link>
+  <joint name="rear_caster_joint" type="fixed">
+    <parent link="base_link"/>
+    <child link="rear_caster_link"/>
+    <!-- 后万向轮位置：底盘后方 -->
+    <origin xyz="-0.15 0 -0.05" rpy="0 0 0"/>
+  </joint>
+  <!-- =========================================================
+       驱动轮定义
     ========================================================== -->
   <xacro:macro name="wheel" params="prefix x_reflect y_reflect">
@@ -197,3 +260,20 @@
     <material>Gazebo/Black</material>
   </gazebo>
+  <!-- 万向轮摩擦力属性（低摩擦，便于转向） -->
+  <gazebo reference="front_caster_link">
+    <mu1>0.0</mu1>  <!-- 万向轮低摩擦 -->
+    <mu2>0.0</mu2>
+    <kp>1000000.0</kp>
+    <kd>100.0</kd>
+    <minDepth>0.001</minDepth>
+    <material>Gazebo/Grey</material>
+  </gazebo>
+  <gazebo reference="rear_caster_link">
+    <mu1>0.0</mu1>  <!-- 万向轮低摩擦 -->
+    <mu2>0.0</mu2>
+    <kp>1000000.0</kp>
+    <kd>100.0</kd>
+    <minDepth>0.001</minDepth>
+    <material>Gazebo/Grey</material>
+  </gazebo>
 </robot>
